File: extrom.kicad_pcb (KiCad board)
At the start: 2 copper layers, 120.2 x 69.7 mm, 78 parts, among them IC1 74HCT00, IC10 74HCT32, IC11 74LS123N, IC12 LM1889N, IC13 2318, IC14 CD4053, IC2 74HCT273, IC3 74HCT20, IC4 74HCT86, IC5 74HCT393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

Commit message: rework pcb
Parts:
- removed U8: 74LS245, Package_DIP:DIP-20_W7.62mm
- added IC23: 74HCT245, Package_SO:SOIC-20W_7.5x12.8mm_P1.27mm, F.Cu at (167.3, 59.8)
- C13: value 22pF -> 4.7pF
- C14: value 4.7pF -> 22pF
- C19, C20, C21, C22, C23: footprint Capacitor_SMD:CP_Elec_6.3x5.8 -> Capacitor_Tantalum_SMD:CP_EIA-3528-21_Kemet-B_Pad1.50x2.35mm_HandSolder; moved to B.Cu
- C2: value 33pF -> 330pF
- C3: value 330pF -> 180pF
- C4: value 180pF -> 100pF
- C5: value 100pF -> 33pF
- C7: value 2-22pF -> 180pF; footprint Dragon:Trimmer-7.5mm -> Capacitor_SMD:C_0805_2012Metric_Pad1.18x1.45mm_HandSolder
- C8: value 33pF -> 2-22pF; footprint Capacitor_SMD:C_0805_2012Metric_Pad1.18x1.45mm_HandSolder -> Dragon:Trimmer-7.5mm
- C9: value 180pF -> 33pF
- IC15: renamed from U1; value 74LS393 -> 74HCT393; footprint Package_DIP:DIP-14_W7.62mm -> Package_SO:SOIC-14_3.9x8.7mm_P1.27mm
- IC16: renamed from U2; value 74LS393 -> 74HCT393; footprint Package_DIP:DIP-14_W7.62mm -> Package_SO:SOIC-14_3.9x8.7mm_P1.27mm
- IC17: renamed from U3; value 74LS04 -> 74HCT04; footprint Package_DIP:DIP-14_W7.62mm -> Package_SO:SOIC-14_3.9x8.7mm_P1.27mm
- IC18: renamed from U4; value 74LS257 -> 74HCT257; footprint Package_DIP:DIP-16_W7.62mm -> Package_SO:SOIC-16_3.9x9.9mm_P1.27mm
- IC19: renamed from U7; value 74LS257 -> 74HCT257; footprint Package_DIP:DIP-16_W7.62mm -> Package_SO:SOIC-16_3.9x9.9mm_P1.27mm
- IC20: renamed from U10; value 74LS257 -> 74HCT257; footprint Package_DIP:DIP-16_W7.62mm -> Package_SO:SOIC-16_3.9x9.9mm_P1.27mm
- IC21: renamed from U9; value 74LS257 -> 74HCT257; footprint Package_DIP:DIP-16_W7.62mm -> Package_SO:SOIC-16_3.9x9.9mm_P1.27mm
- IC22: renamed from U6; value 74LS08 -> 74HCT08; footprint Package_DIP:DIP-14_W7.62mm -> Package_SO:SOIC-14_3.9x8.7mm_P1.27mm
- IC24: renamed from U11; value 74LS02 -> 74HCT02; footprint Package_DIP:DIP-14_W7.62mm -> Package_SO:SOIC-14_3.9x8.7mm_P1.27mm
- IC25: renamed from U12; value 74LS32 -> 74HCT1G32; footprint Package_DIP:DIP-14_W7.62mm -> Package_TO_SOT_SMD:SOT-353_SC-70-5_Handsoldering
- IC26: renamed from U5; footprint Package_DIP:DIP-28_W15.24mm -> Package_DIP:DIP-28_W7.62mm
- J1: value Board Interconnect Male -> Board Interconnect male
- J2: value Video Output -> Video Output male
- R1: value 3K3 -> 27K
- R10: value 22K -> 10K
- R11: value 1K -> 22K
- R12: value 10K -> 1K
- R2: value 1K -> 3K3
- R3: value 5K6 -> 1K
- R4: value 27K -> 5K6
- moved IC18 173.0 mm to (169.0, 88.7), turned to 90 degrees
- moved C19 166.9 mm to (170.3, 51.7), turned to 180 degrees
- moved C22 162.0 mm to (162.9, 87.9), turned to -90 degrees
- moved IC19 150.8 mm to (154.9, 88.7), turned to 90 degrees
- moved C20 150.1 mm to (142.4, 95.1)
- moved C23 146.4 mm to (148.7, 88.0), turned to -90 degrees
- moved C21 139.6 mm to (143.8, 60.5), turned to 180 degrees
- moved C18 139.2 mm to (131.7, 75.9), turned to -90 degrees
- moved IC26 134.3 mm to (139.7, 79.8), turned to 90 degrees
- moved IC21 131.6 mm to (143.2, 88.9), turned to 180 degrees
- moved IC22 121.6 mm to (145.7, 45.1), turned to 90 degrees
- moved IC25 110.7 mm to (154.2, 47.3)
- moved IC20 109.4 mm to (142.6, 64.6)
- moved J3 75.6 mm to (152.3, 53.5), turned to -90 degrees
- moved IC15 64.8 mm to (50.4, 38.9)
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Connections:
- C13 pad 1: MUX X -> Net-(IC13-+)
- C13 pad 2: GND -> Net-(IC14-Z0)
- C14 pad 1: Net-(IC13-+) -> MUX X
- C14 pad 2: (no net) -> GND
- C2 pad 1: LAG -> Net-(IC11A-RCext)
- C3 pad 1: Net-(IC11A-RCext) -> Net-(C3-Pad1)
- C5 pad 1: (no net) -> LAG
- C7 pad 1: (no net) -> GND
- C7 pad 2: -5V -> /VDG/LINE PULSES
- C8 pad 1: Net-(C6-Pad1) -> Net-(C8-Pad1)
- C8 pad 2: (no net) -> -5V
- C9 pad 1: GND -> Net-(C6-Pad1)
- C9 pad 2: (no net) -> Net-(C9-Pad2)
- IC13 pad 6: (no net) -> Net-(IC14-Z0)
- IC2 pad 13: D4 -> DB4
- IC2 pad 14: D5 -> DB5
- IC2 pad 17: D6 -> DB6
- IC2 pad 18: D7 -> DB7
- IC2 pad 3: D0 -> DB0
- IC2 pad 4: D1 -> DB1
- IC2 pad 7: D2 -> DB2
- IC2 pad 8: D3 -> DB3
- IC25 pad 3: INV' -> GND
- IC25 pad 4: unconnected-(U12-Pad4) -> INV'
- IC25 pad 5: unconnected-(U12-Pad5) -> +5V
- J1 pad 11: (no net) -> D4
- J1 pad 13: (no net) -> D5
- J1 pad 15: (no net) -> D6
- J1 pad 17: (no net) -> D7
- J1 pad 3: (no net) -> D0
- J1 pad 5: (no net) -> D1
- J1 pad 7: (no net) -> D2
- J1 pad 9: (no net) -> D3
- R1 pad 1: -5V -> Net-(IC11A-RCext)
- R1 pad 2: ChrOSC -> +5V
- R10 pad 1: Composite -> Net-(IC13-+)
- R10 pad 2: GND -> Net-(IC14-Z0)
- R11 pad 1: MUX X -> Composite
- R11 pad 2: Net-(TR1-B) -> GND
- R12 pad 1: Net-(IC13-+) -> MUX X
- R12 pad 2: (no net) -> Net-(TR1-B)
- R2 pad 1: (no net) -> -5V
- R2 pad 2: LAG -> ChrOSC
- R3 pad 1: (no net) -> Net-(C9-Pad2)
- R3 pad 2: ChrOSC -> LAG
- R4 pad 1: Net-(IC11A-RCext) -> Net-(C8-Pad1)
- R4 pad 2: +5V -> ChrOSC
- R6 pad 2: (no net) -> Net-(IC1-Pad3)
- Y1 pad 1: (no net) -> Net-(C9-Pad2)
- Y1 pad 2: (no net) -> Net-(C8-Pad1)
Routing:
- net +5V: track 161.8 -> 27.8 mm, vias 2 -> 15
- net INV: track 0.00 -> 107.8 mm, vias 0 -> 4
- net ~{RAS0}: track 0.00 -> 95.1 mm, vias 0 -> 1
- net ~{A}/S': track 0.00 -> 90.1 mm, vias 0 -> 2
- net ~{INT}/EXT: track 0.00 -> 88.6 mm, vias 0 -> 3
- net GND: track 127.3 -> 85.9 mm, vias 9 -> 25
- net DA7: track 0.00 -> 38.1 mm, vias 0 -> 4
- net DA4: track 0.00 -> 37.1 mm, vias 0 -> 2
- net DA5: track 0.00 -> 36.6 mm, vias 0 -> 2
- net DC7: track 0.00 -> 33.0 mm
- net DA6: track 0.00 -> 32.4 mm, vias 0 -> 2
- net phiB: track 40.7 -> 71.2 mm
- net ~{A}/S: track 0.00 -> 30.0 mm
- net ~{R}/W: track 0.00 -> 30.0 mm, vias 0 -> 2
- net DC6: track 0.00 -> 29.9 mm
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- added copper zone on In2.Cu, net +5V
- added copper zone on In1.Cu, net GND
Other:
- copper layers 2 -> 4

Commit message: wired board
Parts:
- C2, C3, IC25, J3, R1, R6, R7, R8: moved to B.Cu
- IC10: footprint Package_SO:SOIC-16_3.9x9.9mm_P1.27mm -> Package_SO:SOIC-14_3.9x8.7mm_P1.27mm
- IC2: value 74HCT273 -> 74HC273; footprint Package_SO:TSSOP-20_4.4x6.5mm_P0.65mm -> Package_SO:SO-20_5.3x12.6mm_P1.27mm
- IC23: footprint Package_SO:SOIC-20W_7.5x12.8mm_P1.27mm -> Package_SO:SO-20_5.3x12.6mm_P1.27mm
- moved IC16 118.6 mm to (175.0, 72.7), turned to 90 degrees
- moved IC15 116.5 mm to (162.0, 72.7), turned to 90 degrees
- moved IC4 87.4 mm to (167.1, 135.7)
- moved IC6 80.1 mm to (176.1, 135.7)
- moved C3 76.6 mm to (175.0, 82.5)
- moved IC3 75.7 mm to (133.2, 135.6)
- moved IC7 73.7 mm to (142.0, 135.6)
- moved IC17 69.9 mm to (135.5, 68.3)
- moved R1 62.0 mm to (168.5, 112.0)
- moved IC5 60.0 mm to (124.5, 135.7)
- moved C2 59.7 mm to (168.5, 110.0), turned to 180 degrees
- moved IC24 57.2 mm to (127.0, 85.4)
- moved C20 53.8 mm to (179.4, 56.0)
- moved IC11 49.2 mm to (172.7, 110.9), turned to 90 degrees
- moved IC1 47.6 mm to (175.6, 89.7), turned to 90 degrees
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Connections:
- net Net-(IC2-Q1) renamed /VDG/DV1
- IC17 pad 1: Net-(IC17-Pad1) -> ~{R}/W
- IC17 pad 11: ~{A}/S -> ~{SelInv}
- IC17 pad 12: Net-(IC23-CE) -> Net-(IC26-~{WE})
- IC17 pad 2: SELA -> Net-(IC23-CE)
- IC17 pad 5: ~{SelInv} -> ~{A}/S
- IC17 pad 8: Net-(IC26-~{WE}) -> SELA
- IC17 pad 9: ~{R}/W -> Net-(IC17-Pad9)
- IC18 pad 10: DA7 -> DA4
- IC18 pad 11: D7 -> D4
- IC18 pad 2: D4 -> D7
- IC18 pad 3: DA4 -> DA7
- IC18 pad 4: DB4 -> DB7
- IC18 pad 9: DB7 -> DB4
- IC19 pad 10: DA3 -> DA0
- IC19 pad 11: D3 -> D0
- IC19 pad 2: D0 -> D3
- IC19 pad 3: DA0 -> DA3
- IC19 pad 4: DB0 -> DB3
- IC19 pad 9: DB3 -> DB0
- IC2 pad 12: Net-(IC2-Q4) -> ~{A}/S
- IC2 pad 13: DB4 -> DB7
- IC2 pad 14: DB5 -> DB3
- IC2 pad 15: Net-(IC2-Q5) -> /VDG/DV3
- IC2 pad 16: INV -> /VDG/DV4
- IC2 pad 17: DB6 -> DB4
- IC2 pad 18: DB7 -> DB5
- IC2 pad 19: ~{A}/S -> /VDG/DV5
- IC2 pad 2: Net-(IC2-Q0) -> /VDG/DV2
- IC2 pad 3: DB0 -> DB2
- IC2 pad 6: Net-(IC2-Q2) -> /VDG/DV0
- IC2 pad 7: DB2 -> DB0
- IC2 pad 8: DB3 -> DB6
- IC2 pad 9: Net-(IC2-Q3) -> INV
- IC20 pad 10: AB11 -> AB8
- IC20 pad 11: D7 -> D4
- IC20 pad 2: D4 -> D7
- IC20 pad 3: AB8 -> AB11
- IC20 pad 4: AC8 -> AC11
- IC20 pad 9: AC11 -> AC8
- IC21 pad 10: AB7 -> AB4
- IC21 pad 11: D3 -> D0
- IC21 pad 2: D0 -> D3
- IC21 pad 3: AB4 -> AB7
- IC21 pad 4: AC4 -> AC7
- IC21 pad 9: AC7 -> AC4
- IC22 pad 12: Net-(IC17-Pad6) -> Net-(IC17-Pad10)
- IC22 pad 6: Net-(IC17-Pad1) -> Net-(IC17-Pad9)
- IC23 pad 11: DA7 -> DA0
- IC23 pad 12: DA6 -> DA1
- IC23 pad 13: DA5 -> DA2
- IC23 pad 14: DA4 -> DA3
- IC23 pad 15: DA3 -> DA4
- IC23 pad 16: DA2 -> DA5
- IC23 pad 17: DA1 -> DA6
- IC23 pad 18: DA0 -> DA7
- IC23 pad 2: DC0 -> DC7
- IC23 pad 3: DC1 -> DC6
- IC23 pad 4: DC2 -> DC5
- IC23 pad 5: DC3 -> DC4
- IC23 pad 6: DC4 -> DC3
- IC23 pad 7: DC5 -> DC2
- IC23 pad 8: DC6 -> DC1
- IC23 pad 9: DC7 -> DC0
- IC24 pad 8: Net-(IC17-Pad10) -> Net-(IC17-Pad6)
- IC26 pad 11: DA0 -> DA7
- IC26 pad 12: DA1 -> DA5
- IC26 pad 13: DA2 -> DA3
- IC26 pad 15: DA3 -> DA0
- IC26 pad 16: DA4 -> DA1
- IC26 pad 17: DA5 -> DA2
- IC26 pad 18: DA6 -> DA4
- IC26 pad 19: DA7 -> DA6
- IC8 pad 22: DA0 -> AD0
- IC8 pad 3: Net-(IC2-Q0) -> /VDG/DV0
- IC8 pad 5: Net-(IC2-Q2) -> /VDG/DV2
- IC8 pad 6: Net-(IC2-Q3) -> /VDG/DV3
- IC8 pad 7: Net-(IC2-Q4) -> /VDG/DV4
- IC8 pad 8: Net-(IC2-Q5) -> /VDG/DV5
- J1 pad 6: DA0 -> AD0
- J3 pad 1: DC0 -> Alpha
- J3 pad 10: RC -> DC4
- J3 pad 11: DC5 -> unconnected-(J3-Pin_11-Pad11)
- J3 pad 12: unconnected-(J3-Pin_12-Pad12) -> DC5
- J3 pad 13: DC6 -> unconnected-(J3-Pin_13-Pad13)
- J3 pad 14: unconnected-(J3-Pin_14-Pad14) -> DC6
- J3 pad 15: DC7 -> unconnected-(J3-Pin_15-Pad15)
- J3 pad 16: unconnected-(J3-Pin_16-Pad16) -> DC7
- J3 pad 2: Alpha -> DC0
- J3 pad 3: DC1 -> Inverse
- J3 pad 4: Inverse -> DC1
- J3 pad 5: DC2 -> ~{SelInv}
- J3 pad 6: ~{SelInv} -> DC2
- J3 pad 7: DC3 -> RClk
- J3 pad 8: RClk -> DC3
- J3 pad 9: DC4 -> RC
Routing:
- net +5V: track 27.8 -> 409.5 mm, vias 15 -> 34
- net D2: track 0.00 -> 168.4 mm, vias 0 -> 2
- net D3: track 0.00 -> 167.1 mm, vias 0 -> 2
- net D1: track 0.00 -> 157.4 mm, vias 0 -> 2
- net D0: track 0.00 -> 154.0 mm, vias 0 -> 2
- net D4: track 17.1 -> 165.6 mm, vias 1 -> 2
- net ~{HS}: track 0.00 -> 145.1 mm, vias 0 -> 7
- net D6: track 24.6 -> 168.6 mm, vias 1 -> 2
- net D5: track 20.9 -> 164.4 mm, vias 1 -> 2
- net D7: track 28.8 -> 166.9 mm, vias 1 -> 2
- net ~{FS}: track 0.00 -> 128.9 mm, vias 0 -> 6
- net /VDG/LINE PULSES: track 7.58 -> 135.0 mm, vias 2 -> 8
- net VCLK: track 0.00 -> 112.5 mm, vias 0 -> 5
- net Net-(IC7B-Q1): track 0.00 -> 105.6 mm, vias 0 -> 4
- net Net-(IC7B-Q3): track 0.00 -> 97.4 mm, vias 0 -> 2
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- added copper zone on In1.Cu, net +5V
- added copper zone on In2.Cu, net GND
- removed copper zone on In2.Cu, net +5V
- removed copper zone on In1.Cu, net GND
Other:
- board size 120.2 x 69.7 mm -> 120.2 x 104.1 mm
