File: extrom.kicad_sch (KiCad schematic)
At the start: 19 parts, among them IC10 74HCT32, U1 74LS393, U10 74LS257, U11 74LS02, U12 74LS32, U2 74LS393, U3 74LS04, U4 74LS257, U5 HM62256BLP, U6 74LS08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

Commit message: rework pcb
Parts:
- removed U12: 74LS32, Package_DIP:DIP-14_W7.62mm, symbol 74xx:74LS32
- added IC25: 74HCT1G32, Package_TO_SOT_SMD:SOT-353_SC-70-5_Handsoldering, symbol 74xGxx:74AHCT1G32
- C1: footprint Capacitor_SMD:CP_Elec_6.3x5.8 -> Capacitor_Tantalum_SMD:CP_EIA-3528-21_Kemet-B_Pad1.50x2.35mm_HandSolder
- IC15: renamed from U1; value 74LS393 -> 74HCT393; footprint Package_DIP:DIP-14_W7.62mm -> Package_SO:SOIC-14_3.9x8.7mm_P1.27mm
- IC16: renamed from U2; value 74LS393 -> 74HCT393; footprint Package_DIP:DIP-14_W7.62mm -> Package_SO:SOIC-14_3.9x8.7mm_P1.27mm
- IC17: renamed from U3; value 74LS04 -> 74HCT04; footprint Package_DIP:DIP-14_W7.62mm -> Package_SO:SOIC-14_3.9x8.7mm_P1.27mm
- IC18: renamed from U4; value 74LS257 -> 74HCT257; footprint Package_DIP:DIP-16_W7.62mm -> Package_SO:SOIC-16_3.9x9.9mm_P1.27mm
- IC19: renamed from U7; value 74LS257 -> 74HCT257; footprint Package_DIP:DIP-16_W7.62mm -> Package_SO:SOIC-16_3.9x9.9mm_P1.27mm
- IC20: renamed from U10; value 74LS257 -> 74HCT257; footprint Package_DIP:DIP-16_W7.62mm -> Package_SO:SOIC-16_3.9x9.9mm_P1.27mm
- IC21: renamed from U9; value 74LS257 -> 74HCT257; footprint Package_DIP:DIP-16_W7.62mm -> Package_SO:SOIC-16_3.9x9.9mm_P1.27mm
- IC22: renamed from U6; value 74LS08 -> 74HCT08; footprint Package_DIP:DIP-14_W7.62mm -> Package_SO:SOIC-14_3.9x8.7mm_P1.27mm
- IC23: renamed from U8; value 74LS245 -> 74HCT245; footprint Package_DIP:DIP-20_W7.62mm -> Package_SO:SOIC-20W_7.5x12.8mm_P1.27mm
- IC24: renamed from U11; value 74LS02 -> 74HCT02; footprint Package_DIP:DIP-14_W7.62mm -> Package_SO:SOIC-14_3.9x8.7mm_P1.27mm
- IC26: renamed from U5; footprint Package_DIP:DIP-28_W15.24mm -> Package_DIP:DIP-28_W7.62mm
Connections:
- net +5V: now also IC25.5 (VCC)
- net GND: now also IC25.3 (GND)
- net INV': now also IC25.4
- net at IC22.8: now also IC25.1
- net at IC22.11: now also IC25.2
- no-connect marks 12 -> 3
Other:
- note added: "Databus B (internal or external data)"
- note added: "Databus a (external data)"
- note added: "select data bus A or main"
- note removed: "select internal or external data"

Commit message: wired board
Parts:
- IC10: footprint Package_SO:SOIC-16_3.9x9.9mm_P1.27mm -> Package_SO:SOIC-14_3.9x8.7mm_P1.27mm
- IC23: footprint Package_SO:SOIC-20W_7.5x12.8mm_P1.27mm -> Package_SO:SO-20_5.3x12.6mm_P1.27mm
Connections:
- net AB11: now also IC20.3 (I1a); no longer IC20.10 (I1d)
- net AB4: now also IC21.10 (I1d); no longer IC21.3 (I1a)
- net AB7: now also IC21.3 (I1a); no longer IC21.10 (I1d)
- net AB8: now also IC20.10 (I1d); no longer IC20.3 (I1a)
- net AC11: now also IC20.4 (Za); no longer IC20.9 (Zd)
- net AC4: now also IC21.9 (Zd); no longer IC21.4 (Za)
- net AC7: now also IC21.4 (Za); no longer IC21.9 (Zd)
- net AC8: now also IC20.9 (Zd); no longer IC20.4 (Za)
- net D0: now also IC19.11 (I0d), IC21.11 (I0d); no longer IC19.2 (I0a), IC21.2 (I0a)
- net D3: now also IC19.2 (I0a), IC21.2 (I0a); no longer IC19.11 (I0d), IC21.11 (I0d)
- net D4: now also IC18.11 (I0d), IC20.11 (I0d); no longer IC18.2 (I0a), IC20.2 (I0a)
- net D7: now also IC18.2 (I0a), IC20.2 (I0a); no longer IC18.11 (I0d), IC20.11 (I0d)
- net DA0: now also IC19.10 (I1d), IC23.11 (B7), IC26.15 (Q3); no longer IC19.3 (I1a), IC23.18 (B0), IC26.11 (Q0)
- net DA1: now also IC23.12 (B6), IC26.16 (Q4); no longer IC23.17 (B1), IC26.12 (Q1)
- net DA2: now also IC23.13 (B5), IC26.17 (Q5); no longer IC23.16 (B2), IC26.13 (Q2)
- net DA3: now also IC19.3 (I1a), IC23.14 (B4), IC26.13 (Q2); no longer IC19.10 (I1d), IC23.15 (B3), IC26.15 (Q3)
- net DA4: now also IC18.10 (I1d), IC23.15 (B3), IC26.18 (Q6); no longer IC18.3 (I1a), IC23.14 (B4), IC26.16 (Q4)
- net DA5: now also IC23.16 (B2), IC26.12 (Q1); no longer IC23.13 (B5), IC26.17 (Q5)
- net DA6: now also IC23.17 (B1), IC26.19 (Q7); no longer IC23.12 (B6), IC26.18 (Q6)
- net DA7: now also IC18.3 (I1a), IC23.18 (B0), IC26.11 (Q0); no longer IC18.10 (I1d), IC23.11 (B7), IC26.19 (Q7)
- net DB0: now also IC19.9 (Zd); no longer IC19.4 (Za)
- net DB3: now also IC19.4 (Za); no longer IC19.9 (Zd)
- net DB4: now also IC18.9 (Zd); no longer IC18.4 (Za)
- net DB7: now also IC18.4 (Za); no longer IC18.9 (Zd)
- net DC0: now also IC23.9 (A7); no longer IC23.2 (A0)
- net DC1: now also IC23.8 (A6); no longer IC23.3 (A1)
- net DC2: now also IC23.7 (A5); no longer IC23.4 (A2)
- net DC3: now also IC23.6 (A4); no longer IC23.5 (A3)
- net DC4: now also IC23.5 (A3); no longer IC23.6 (A4)
- net DC5: now also IC23.4 (A2); no longer IC23.7 (A5)
- net DC6: now also IC23.3 (A1); no longer IC23.8 (A6)
- net DC7: now also IC23.2 (A0); no longer IC23.9 (A7)
- net SELA: now also IC17.8; no longer IC17.2
- net ~{A}/S: now also IC17.5; no longer IC17.11
- net ~{R}/W: now also IC17.1, IC17.13; no longer IC17.13, IC17.9
- net ~{SelInv}: now also IC17.11; no longer IC17.5
- net at IC23.19 (CE): now also IC17.2; no longer IC17.12
- net at IC22.12: now also IC17.10; no longer IC17.6
- net at IC24.8: now also IC17.6; no longer IC17.10
- net at IC26.27 (~{WE}): now also IC17.12; no longer IC17.8
- net at IC22.6: now also IC17.9; no longer IC17.1
