File: interface.kicad_sch (KiCad schematic)
At the start: 3 parts, among them J2 Board Interconnect male, J2 Video Output male, J3 Conn_02x08_Odd_Even

Commit message: wired board
Connections:
- net Alpha: now also J3.1 (Pin_1); no longer J3.2 (Pin_2)
- net DC0: now also J3.2 (Pin_2); no longer J3.1 (Pin_1)
- net DC1: now also J3.4 (Pin_4); no longer J3.3 (Pin_3)
- net DC2: now also J3.6 (Pin_6); no longer J3.5 (Pin_5)
- net DC3: now also J3.8 (Pin_8); no longer J3.7 (Pin_7)
- net DC4: now also J3.10 (Pin_10); no longer J3.9 (Pin_9)
- net DC5: now also J3.12 (Pin_12); no longer J3.11 (Pin_11)
- net DC6: now also J3.14 (Pin_14); no longer J3.13 (Pin_13)
- net DC7: now also J3.16 (Pin_16); no longer J3.15 (Pin_15)
- net Inverse: now also J3.3 (Pin_3); no longer J3.4 (Pin_4)
- net RC: now also J3.9 (Pin_9); no longer J3.10 (Pin_10)
- net RClk: now also J3.7 (Pin_7); no longer J3.8 (Pin_8)
- net ~{SelInv}: now also J3.5 (Pin_5); no longer J3.6 (Pin_6)
- net DA0 renamed AD0
Changed lines of the file:
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@@
     (date "2023-07-31")
   )
+  (no_connect (at 58.42 107.95))
   (no_connect (at 58.42 74.93))
-  (no_connect (at 71.12 107.95))
-  (no_connect (at 71.12 105.41))
+  (no_connect (at 58.42 105.41))
+  (no_connect (at 58.42 102.87))
   (no_connect (at 101.6508 53.0352))
-  (no_connect (at 71.12 102.87))
-  (global_label "DC1" (shape input) (at 58.42 92.71 180) (fields_autoplaced)
-    (effects (font (size 1.27 1.27)) (justify right))
-    (property "Intersheetrefs" "${INTERSHEET_REFS}" (at 51.7647 92.71 0)
-      (effects (font (size 1.27 1.27)) (justify right) hide)
-    )
-  )
   (global_label "VID OUT" (shape output) (at 101.6508 55.5752 0) (fields_autoplaced)
     (effects (font (size 1.27 1.27)) (justify left))
@@
     )
   )
-  (global_label "DC7" (shape input) (at 58.42 107.95 180) (fields_autoplaced)
+  (global_label "~{SelInv}" (shape input) (at 58.42 95.25 180) (fields_autoplaced)
     (effects (font (size 1.27 1.27)) (justify right))
-    (property "Intersheetrefs" "${INTERSHEET_REFS}" (at 51.7647 107.95 0)
+    (property "Intersheetrefs" "${INTERSHEET_REFS}" (at 49.7501 95.25 0)
       (effects (font (size 1.27 1.27)) (justify right) hide)
     )
   )
-  (global_label "DA0" (shape output) (at 71.12 54.61 0) (fields_autoplaced)
+  (global_label "RC" (shape input) (at 58.42 100.33 180) (fields_autoplaced)
+    (effects (font (size 1.27 1.27)) (justify right))
+    (property "Intersheetrefs" "${INTERSHEET_REFS}" (at 52.9742 100.33 0)
+      (effects (font (size 1.27 1.27)) (justify right) hide)
+    )
+  )
+  (global_label "DC4" (shape input) (at 71.12 100.33 0) (fields_autoplaced)
     (effects (font (size 1.27 1.27)) (justify left))
-    (property "Intersheetrefs" "${INTERSHEET_REFS}" (at 76.9397 54.61 0)
+    (property "Intersheetrefs" "${INTERSHEET_REFS}" (at 77.7753 100.33 0)
+      (effects (font (size 1.27 1.27)) (justify left) hide)
+    )
+  )
+  (global_label "AD0" (shape output) (at 71.12 54.61 0) (fields_autoplaced)
+    (effects (font (size 1.27 1.27)) (justify left))
+    (property "Intersheetrefs" "${INTERSHEET_REFS}" (at 77.6733 54.61 0)
       (effects (font (size 1.27 1.27)) (justify left) hide)
     )
@@
     )
   )
+  (global_label "RClk" (shape input) (at 58.42 97.79 180) (fields_autoplaced)
+    (effects (font (size 1.27 1.27)) (justify right))
+    (property "Intersheetrefs" "${INTERSHEET_REFS}" (at 51.2809 97.79 0)
+      (effects (font (size 1.27 1.27)) (justify right) hide)
+    )
+  )
   (global_label "~{NHS}" (shape output) (at 71.12 57.15 0) (fields_autoplaced)
     (effects (font (size 1.27 1.27)) (justify left))
     (property "Intersheetrefs" "${INTERSHEET_REFS}" (at 77.2421 57.15 0)
+      (effects (font (size 1.27 1.27)) (justify left) hide)
+    )
+  )
+  (global_label "DC0" (shape input) (at 71.12 90.17 0) (fields_autoplaced)
+    (effects (font (size 1.27 1.27)) (justify left))
+    (property "Intersheetrefs" "${INTERSHEET_REFS}" (at 77.7753 90.17 0)
       (effects (font (size 1.27 1.27)) (justify left) hide)
     )
@@
     )
   )
-  (global_label "Alpha" (shape input) (at 71.12 90.17 0) (fields_autoplaced)
+  (global_label "DC3" (shape input) (at 71.12 97.79 0) (fields_autoplaced)
     (effects (font (size 1.27 1.27)) (justify left))
-    (property "Intersheetrefs" "${INTERSHEET_REFS}" (at 79.306 90.17 0)
+    (property "Intersheetrefs" "${INTERSHEET_REFS}" (at 77.7753 97.79 0)
       (effects (font (size 1.27 1.27)) (justify left) hide)
     )
@@
     )
   )
-  (global_label "DC3" (shape input) (at 58.42 97.79 180) (fields_autoplaced)
+  (global_label "Alpha" (shape input) (at 58.42 90.17 180) (fields_autoplaced)
     (effects (font (size 1.27 1.27)) (justify right))
-    (property "Intersheetrefs" "${INTERSHEET_REFS}" (at 51.7647 97.79 0)
+    (property "Intersheetrefs" "${INTERSHEET_REFS}" (at 50.234 90.17 0)
       (effects (font (size 1.27 1.27)) (justify right) hide)
     )
@@
     )
   )
-  (global_label "Inverse" (shape input) (at 71.12 92.71 0) (fields_autoplaced)
-    (effects (font (size 1.27 1.27)) (justify left))
-    (property "Intersheetrefs" "${INTERSHEET_REFS}" (at 80.8181 92.71 0)
-      (effects (font (size 1.27 1.27)) (justify left) hide)
-    )
-  )
-  (global_label "RC" (shape input) (at 71.12 100.33 0) (fields_autoplaced)
-    (effects (font (size 1.27 1.27)) (justify left))
-    (property "Intersheetrefs" "${INTERSHEET_REFS}" (at 76.5658 100.33 0)
-      (effects (font (size 1.27 1.27)) (justify left) hide)
-    )
-  )
-  (global_label "RClk" (shape input) (at 71.12 97.79 0) (fields_autoplaced)
-    (effects (font (size 1.27 1.27)) (justify left))
-    (property "Intersheetrefs" "${INTERSHEET_REFS}" (at 78.2591 97.79 0)
-      (effects (font (size 1.27 1.27)) (justify left) hide)
-    )
-  )
-  (global_label "DC4" (shape input) (at 58.42 100.33 180) (fields_autoplaced)
-    (effects (font (size 1.27 1.27)) (justify right))
-    (property "Intersheetrefs" "${INTERSHEET_REFS}" (at 51.7647 100.33 0)
-      (effects (font (size 1.27 1.27)) (justify right) hide)
-    )
-  )
-  (global_label "DC6" (shape input) (at 58.42 105.41 180) (fields_autoplaced)
-    (effects (font (size 1.27 1.27)) (justify right))
-    (property "Intersheetrefs" "${INTERSHEET_REFS}" (at 51.7647 105.41 0)
-      (effects (font (size 1.27 1.27)) (justify right) hide)
-    )
-  )
   (global_label "BIAS" (shape output) (at 101.6508 47.9552 0) (fields_autoplaced)
     (effects (font (size 1.27 1.27)) (justify left))
@@
     )
   )
-  (global_label "~{SelInv}" (shape input) (at 71.12 95.25 0) (fields_autoplaced)
+  (global_label "DC6" (shape input) (at 71.12 105.41 0) (fields_autoplaced)
     (effects (font (size 1.27 1.27)) (justify left))
-    (property "Intersheetrefs" "${INTERSHEET_REFS}" (at 79.7899 95.25 0)
+    (property "Intersheetrefs" "${INTERSHEET_REFS}" (at 77.7753 105.41 0)
       (effects (font (size 1.27 1.27)) (justify left) hide)
     )
@@
     )
   )
-  (global_label "DC0" (shape input) (at 58.42 90.17 180) (fields_autoplaced)
-    (effects (font (size 1.27 1.27)) (justify right))
-    (property "Intersheetrefs" "${INTERSHEET_REFS}" (at 51.7647 90.17 0)
-      (effects (font (size 1.27 1.27)) (justify right) hide)
+  (global_label "DC2" (shape input) (at 71.12 95.25 0) (fields_autoplaced)
+    (effects (font (size 1.27 1.27)) (justify left))
+    (property "Intersheetrefs" "${INTERSHEET_REFS}" (at 77.7753 95.25 0)
+      (effects (font (size 1.27 1.27)) (justify left) hide)
     )
   )
@@
     )
   )
-  (global_label "DC2" (shape input) (at 58.42 95.25 180) (fields_autoplaced)
-    (effects (font (size 1.27 1.27)) (justify right))
-    (property "Intersheetrefs" "${INTERSHEET_REFS}" (at 51.7647 95.25 0)
-      (effects (font (size 1.27 1.27)) (justify right) hide)
-    )
-  )
   (global_label "D3" (shape input) (at 58.42 59.69 180) (fields_autoplaced)
     (effects (font (size 1.27 1.27)) (justify right))
     (property "Intersheetrefs" "${INTERSHEET_REFS}" (at 52.9553 59.69 0)
       (effects (font (size 1.27 1.27)) (justify right) hide)
+    )
+  )
+  (global_label "DC7" (shape input) (at 71.12 107.95 0) (fields_autoplaced)
+    (effects (font (size 1.27 1.27)) (justify left))
+    (property "Intersheetrefs" "${INTERSHEET_REFS}" (at 77.7753 107.95 0)
+      (effects (font (size 1.27 1.27)) (justify left) hide)
     )
   )
@@
     )
   )
+  (global_label "DC5" (shape input) (at 71.12 102.87 0) (fields_autoplaced)
+    (effects (font (size 1.27 1.27)) (justify left))
+    (property "Intersheetrefs" "${INTERSHEET_REFS}" (at 77.7753 102.87 0)
+      (effects (font (size 1.27 1.27)) (justify left) hide)
+    )
+  )
   (global_label "D2" (shape input) (at 58.42 57.15 180) (fields_autoplaced)
     (effects (font (size 1.27 1.27)) (justify right))
@@
     )
   )
-  (global_label "DC5" (shape input) (at 58.42 102.87 180) (fields_autoplaced)
+  (global_label "Inverse" (shape input) (at 58.42 92.71 180) (fields_autoplaced)
     (effects (font (size 1.27 1.27)) (justify right))
-    (property "Intersheetrefs" "${INTERSHEET_REFS}" (at 51.7647 102.87 0)
+    (property "Intersheetrefs" "${INTERSHEET_REFS}" (at 48.7219 92.71 0)
       (effects (font (size 1.27 1.27)) (justify right) hide)
     )
   )
+  (global_label "DC1" (shape input) (at 71.12 92.71 0) (fields_autoplaced)
+    (effects (font (size 1.27 1.27)) (justify left))
+    (property "Intersheetrefs" "${INTERSHEET_REFS}" (at 77.7753 92.71 0)
+      (effects (font (size 1.27 1.27)) (justify left) hide)
+    )
+  )
