File: vdg.kicad_sch (KiCad schematic)
At the start: 58 parts, among them IC1 74HCT273, IC10 74HCT32, IC11 74LS123N, IC12 LM1889N, IC13 2318, IC15 CD4053, IC2 MC6847, IC3 74HCT00, IC4 74HCT20, IC5 74HCT86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

Commit message: rework pcb
Connections:
- net D0 renamed DB0
- net D1 renamed DB1
- net D2 renamed DB2
- net D3 renamed DB3
- net D4 renamed DB4
- net D5 renamed DB5
- net D6 renamed DB6
- net D7 renamed DB7
Other:
- note added: "Databus B (internal or external data)"
Changed lines of the file:
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@@
+    (effects (font (size 1.27 1.27)) (justify left bottom))
+  )
+  (text "Databus B\n(internal or \nexternal data)" (at 16.51 26.67 0)
     (effects (font (size 1.27 1.27)) (justify left bottom))
   )
@@
     (effects (font (size 1.27 1.27)) (justify left bottom))
   )
-  (global_label "D0" (shape input) (at 26.67 30.226 180) (fields_autoplaced)
-    (effects (font (size 1.27 1.27)) (justify right))
-    (property "Intersheetrefs" "${INTERSHEET_REFS}" (at 21.2053 30.226 0)
+  (global_label "DB0" (shape input) (at 26.67 30.226 180) (fields_autoplaced)
+    (effects (font (size 1.27 1.27)) (justify right))
+    (property "Intersheetrefs" "${INTERSHEET_REFS}" (at 19.9353 30.226 0)
       (effects (font (size 1.27 1.27)) (justify right) hide)
     )
@@
     )
   )
-  (global_label "D6" (shape input) (at 26.67 45.466 180) (fields_autoplaced)
-    (effects (font (size 1.27 1.27)) (justify right))
-    (property "Intersheetrefs" "${INTERSHEET_REFS}" (at 21.2053 45.466 0)
+  (global_label "DB6" (shape input) (at 26.67 45.466 180) (fields_autoplaced)
+    (effects (font (size 1.27 1.27)) (justify right))
+    (property "Intersheetrefs" "${INTERSHEET_REFS}" (at 19.9353 45.466 0)
       (effects (font (size 1.27 1.27)) (justify right) hide)
     )
@@
     )
   )
-  (global_label "D7" (shape input) (at 26.67 48.006 180) (fields_autoplaced)
-    (effects (font (size 1.27 1.27)) (justify right))
-    (property "Intersheetrefs" "${INTERSHEET_REFS}" (at 21.2053 48.006 0)
-      (effects (font (size 1.27 1.27)) (justify right) hide)
-    )
-  )
-  (global_label "D1" (shape input) (at 26.67 32.766 180) (fields_autoplaced)
-    (effects (font (size 1.27 1.27)) (justify right))
-    (property "Intersheetrefs" "${INTERSHEET_REFS}" (at 21.2053 32.766 0)
+  (global_label "DB7" (shape input) (at 26.67 48.006 180) (fields_autoplaced)
+    (effects (font (size 1.27 1.27)) (justify right))
+    (property "Intersheetrefs" "${INTERSHEET_REFS}" (at 19.9353 48.006 0)
+      (effects (font (size 1.27 1.27)) (justify right) hide)
+    )
+  )
+  (global_label "DB1" (shape input) (at 26.67 32.766 180) (fields_autoplaced)
+    (effects (font (size 1.27 1.27)) (justify right))
+    (property "Intersheetrefs" "${INTERSHEET_REFS}" (at 19.9353 32.766 0)
       (effects (font (size 1.27 1.27)) (justify right) hide)
     )
@@
     )
   )
-  (global_label "D5" (shape input) (at 26.67 42.926 180) (fields_autoplaced)
-    (effects (font (size 1.27 1.27)) (justify right))
-    (property "Intersheetrefs" "${INTERSHEET_REFS}" (at 21.2053 42.926 0)
+  (global_label "DB5" (shape input) (at 26.67 42.926 180) (fields_autoplaced)
+    (effects (font (size 1.27 1.27)) (justify right))
+    (property "Intersheetrefs" "${INTERSHEET_REFS}" (at 19.9353 42.926 0)
       (effects (font (size 1.27 1.27)) (justify right) hide)
     )
@@
     )
   )
-  (global_label "D3" (shape input) (at 26.67 37.846 180) (fields_autoplaced)
-    (effects (font (size 1.27 1.27)) (justify right))
-    (property "Intersheetrefs" "${INTERSHEET_REFS}" (at 21.2053 37.846 0)
+  (global_label "DB3" (shape input) (at 26.67 37.846 180) (fields_autoplaced)
+    (effects (font (size 1.27 1.27)) (justify right))
+    (property "Intersheetrefs" "${INTERSHEET_REFS}" (at 19.9353 37.846 0)
       (effects (font (size 1.27 1.27)) (justify right) hide)
     )
@@
     )
   )
-  (global_label "D4" (shape input) (at 26.67 40.386 180) (fields_autoplaced)
-    (effects (font (size 1.27 1.27)) (justify right))
-    (property "Intersheetrefs" "${INTERSHEET_REFS}" (at 21.2053 40.386 0)
+  (global_label "DB4" (shape input) (at 26.67 40.386 180) (fields_autoplaced)
+    (effects (font (size 1.27 1.27)) (justify right))
+    (property "Intersheetrefs" "${INTERSHEET_REFS}" (at 19.9353 40.386 0)
       (effects (font (size 1.27 1.27)) (justify right) hide)
     )
@@
     )
   )
-  (global_label "D2" (shape input) (at 26.67 35.306 180) (fields_autoplaced)
-    (effects (font (size 1.27 1.27)) (justify right))
-    (property "Intersheetrefs" "${INTERSHEET_REFS}" (at 21.2053 35.306 0)
+  (global_label "DB2" (shape input) (at 26.67 35.306 180) (fields_autoplaced)
+    (effects (font (size 1.27 1.27)) (justify right))
+    (property "Intersheetrefs" "${INTERSHEET_REFS}" (at 19.9353 35.306 0)
       (effects (font (size 1.27 1.27)) (justify right) hide)
     )
@@
   )
   (symbol (lib_id "Device:C_Trim_Differential") (at 175.26 95.504 0) (unit 1)
-    (in_bom yes) (on_board yes) (dnp no) (fields_autoplaced)
+    (in_bom yes) (on_board yes) (dnp no)
     (property "Reference" "C7" (at 180.848 94.1069 0)
       (effects (font (size 1.27 1.27)) (justify left))

Commit message: wired board
Parts:
- IC1: value 74HCT273 -> 74HC273; footprint Package_SO:TSSOP-20_4.4x6.5mm_P0.65mm -> Package_SO:SO-20_5.3x12.6mm_P1.27mm
- IC10: footprint Package_SO:SOIC-16_3.9x9.9mm_P1.27mm -> Package_SO:SOIC-14_3.9x8.7mm_P1.27mm
Connections:
- net DB0: now also IC1.7 (D2); no longer IC1.3 (D0)
- net DB2: now also IC1.3 (D0); no longer IC1.7 (D2)
- net DB3: now also IC1.14 (D5); no longer IC1.8 (D3)
- net DB4: now also IC1.17 (D6); no longer IC1.13 (D4)
- net DB5: now also IC1.18 (D7); no longer IC1.14 (D5)
- net DB6: now also IC1.8 (D3); no longer IC1.17 (D6)
- net DB7: now also IC1.13 (D4); no longer IC1.18 (D7)
- net INV: now also IC1.9 (Q3); no longer IC1.16 (Q6)
- net ~{A}/S: now also IC1.12 (Q4); no longer IC1.19 (Q7)
- net DV4: now reaches IC2.7 (D4)
- net DV4: now also IC1.16 (Q6); no longer IC1.12 (Q4)
- net DV3: now reaches IC1.15 (Q5)
- net DV3: now also IC2.6 (D3); no longer IC2.8 (D5)
- net DV0: now reaches IC2.3 (D0)
- net DV0: now also IC1.6 (Q2); no longer IC1.2 (Q0)
- net DV1: now reaches IC1.5 (Q1), IC2.4 (D1)
- net DV2: now reaches IC2.5 (D2)
- net DV2: now also IC1.2 (Q0); no longer IC1.6 (Q2)
- net DA0 renamed AD0
- new net DV5: IC1.19 (Q7), IC2.8 (D5)
